File: Circuit/generic_microwave_oven_controller/Soft_Starter.kicad_sch (KiCad schematic)
At the start: 20 parts, among them J1 Screw_Terminal_01x02, J2 AC_IN, J3 AC_OUT, Q1 BT139-600, U1 PC817, U2 MOC3021M

Commit message: :recket: Tested and deploy to board.
Parts:
- removed C1: 0.05u, symbol Device:C
- removed C2: 0.01u, symbol Device:C
- removed R7: 39_1W, symbol Device:R
- R1: value 1k_W25 -> 360_1W
- R4: value 330_W25 -> 220_W25
- R6: value 470_1W -> 360_1W
Connections:
- net ZCD_DC_OUT_M: no longer R2.2
- net ZCD_DC_OUT_P: now also R2.1; no longer R1.1
- net at R6.1: now also R1.2; no longer R5.2
- new net: R2.2, U1.1
- new net: R1.1, R5.2
Other:
- moved on the sheet: Q1, R2
